File: timing_sipm_amp_ufl.kicad_pcb (KiCad board)
At the start: 2 copper layers, 42 x 10 mm, 20 parts, among them J1 HV, J2 Amp, J3 Signal, Q1 BFR92, Q2 PNP

Commit message: Add files via upload
Routing:
- net GND2: track 6.38 -> 4.30 mm, vias 8 -> 14
Changed lines of the file:
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@@
     (property "Sheetname" "")
     (attr smd)
-    (fp_text reference "J1" (at -0.635 -4.445 -90) (layer "F.SilkS")
-      (effects (font (size 1 1) (thickness 0.15)))
-    )
-    (fp_text value "HV" (at 6.35 4.445 -90) (layer "F.Fab")
+    (fp_text reference "J1" (at -0.635 -4.445 -90) (layer "F.Fab")
+      (effects (font (size 1 1) (thickness 0.15)))
+    )
+    (fp_text value "HV" (at -4.315 0.705) (layer "F.SilkS")
       (effects (font (size 1 1) (thickness 0.15)))
     )
@@
     (property "Sheetname" "")
     (attr smd)
-    (fp_text reference "R5" (at 0 -1.17 90) (layer "F.SilkS")
+    (fp_text reference "R5" (at 0 -1.17 90) (layer "F.Fab")
       (effects (font (size 1 1) (thickness 0.15)))
     )
@@
     (property "Sheetname" "")
     (attr smd)
-    (fp_text reference "C5" (at 0 -1.16) (layer "F.SilkS")
+    (fp_text reference "C5" (at 0 -1.16) (layer "F.Fab")
       (effects (font (size 1 1) (thickness 0.15)))
     )
@@
     (property "Sheetname" "")
     (attr smd)
-    (fp_text reference "Q2" (at 0 -2.4) (layer "F.SilkS")
+    (fp_text reference "Q2" (at 0 -2.4) (layer "F.Fab")
       (effects (font (size 1 1) (thickness 0.15)))
     )
@@
     (property "Sheetname" "")
     (attr smd)
-    (fp_text reference "R4" (at 0 -1.17) (layer "F.SilkS")
+    (fp_text reference "R4" (at 0 -1.17) (layer "F.Fab")
       (effects (font (size 1 1) (thickness 0.15)))
     )
@@
     (property "Sheetname" "")
     (attr smd)
-    (fp_text reference "J2" (at 0.475 -3.2 90) (layer "F.SilkS")
-      (effects (font (size 1 1) (thickness 0.15)))
-    )
-    (fp_text value "Amp" (at 0.475 3.2 90) (layer "F.Fab")
+    (fp_text reference "J2" (at 0.475 -3.2 90) (layer "F.Fab")
+      (effects (font (size 1 1) (thickness 0.15)))
+    )
+    (fp_text value "Amp" (at 0.09 -3.18 90) (layer "F.SilkS")
       (effects (font (size 1 1) (thickness 0.15)))
     )
@@
     (property "Sheetname" "")
     (attr smd)
-    (fp_text reference "C1" (at 0 -1.16) (layer "F.SilkS")
+    (fp_text reference "C1" (at 0 -1.16) (layer "F.Fab")
       (effects (font (size 1 1) (thickness 0.15)))
     )
@@
     (property "Sheetname" "")
     (attr smd)
-    (fp_text reference "C2" (at 0 -1.16) (layer "F.SilkS")
+    (fp_text reference "C2" (at 0 -1.16) (layer "F.Fab")
       (effects (font (size 1 1) (thickness 0.15)))
     )
@@
     (property "Sheetname" "")
     (attr smd)
-    (fp_text reference "C4" (at 0 -1.16) (layer "F.SilkS")
+    (fp_text reference "C4" (at 0 -1.16) (layer "F.Fab")
       (effects (font (size 1 1) (thickness 0.15)))
     )
@@
     (property "Sheetname" "")
     (attr smd)
-    (fp_text reference "J3" (at 0.475 -3.2 90) (layer "F.SilkS")
-      (effects (font (size 1 1) (thickness 0.15)))
-    )
-    (fp_text value "Signal" (at 0.475 3.2 90) (layer "F.Fab")
+    (fp_text reference "J3" (at 0.475 -3.2 90) (layer "F.Fab")
+      (effects (font (size 1 1) (thickness 0.15)))
+    )
+    (fp_text value "Signal" (at 0.095 3.155 90) (layer "F.SilkS")
       (effects (font (size 1 1) (thickness 0.15)))
     )
@@
     (property "Sheetname" "")
     (attr smd)
-    (fp_text reference "C3" (at 0 -1.16) (layer "F.SilkS")
+    (fp_text reference "C3" (at 0 -1.16) (layer "F.Fab")
       (effects (font (size 1 1) (thickness 0.15)))
     )
@@
     (property "Sheetname" "")
     (attr smd)
-    (fp_text reference "R7" (at 0 -1.17) (layer "F.SilkS")
+    (fp_text reference "R7" (at 0 -1.17) (layer "F.Fab")
       (effects (font (size 1 1) (thickness 0.15)))
     )
@@
     (property "Sheetname" "")
     (attr smd)
-    (fp_text reference "R2" (at 0 -1.65 90) (layer "F.SilkS")
+    (fp_text reference "R2" (at 0 -1.65 90) (layer "F.Fab")
       (effects (font (size 1 1) (thickness 0.15)))
     )
@@
     (property "Sheetname" "")
     (attr through_hole)
-    (fp_text reference "D1" (at 0 -2.33 90) (layer "F.SilkS")
+    (fp_text reference "D1" (at 0 -2.33 90) (layer "F.Fab")
       (effects (font (size 1 1) (thickness 0.15)))
     )
@@
     (property "Sheetname" "")
     (attr smd)
-    (fp_text reference "R6" (at 0 -1.17) (layer "F.SilkS")
+    (fp_text reference "R6" (at 0 -1.17) (layer "F.Fab")
       (effects (font (size 1 1) (thickness 0.15)))
     )
@@
     (property "Sheetname" "")
     (attr exclude_from_pos_files)
-    (fp_text reference "H2" (at 0 -3.8) (layer "F.SilkS")
+    (fp_text reference "H2" (at 0 -3.8) (layer "F.Fab")
       (effects (font (size 1 1) (thickness 0.15)))
     )
@@
     (property "Sheetname" "")
     (attr smd)
-    (fp_text reference "Q1" (at 0 -2.4) (layer "F.SilkS")
+    (fp_text reference "Q1" (at 0 -2.4) (layer "F.Fab")
       (effects (font (size 1 1) (thickness 0.15)))
     )
@@
     (property "Sheetname" "")
     (attr smd)
-    (fp_text reference "R3" (at 0 -1.17 90) (layer "F.SilkS")
+    (fp_text reference "R3" (at 0 -1.17 90) (layer "F.Fab")
       (effects (font (size 1 1) (thickness 0.15)))
     )
@@
     (property "Sheetname" "")
     (attr smd)
-    (fp_text reference "R1" (at 0 -1.65 180) (layer "F.SilkS")
+    (fp_text reference "R1" (at 0 -1.65 180) (layer "F.Fab")
       (effects (font (size 1 1) (thickness 0.15)))
     )
@@
     (property "Sheetname" "")
     (attr exclude_from_pos_files)
-    (fp_text reference "H1" (at 0 -3.8) (layer "F.SilkS")
+    (fp_text reference "H1" (at 0 -3.8) (layer "F.Fab")
       (effects (font (size 1 1) (thickness 0.15)))
     )
@@
   (segment (start 100.64 71.24) (end 100.67 71.27) (width 0.25) (layer "F.Cu") (net 5))
   (segment (start 98.61 71.2) (end 99.57 71.2) (width 0.25) (layer "F.Cu") (net 5))
-  (segment (start 103.59 70.28) (end 104.75 70.28) (width 0.25) (layer "F.Cu") (net 6))
   (segment (start 95.32 75.69) (end 94.91 75.28) (width 0.25) (layer "F.Cu") (net 6))
   (segment (start 97.64 71.21) (end 97.65 71.2) (width 0.25) (layer "F.Cu") (net 6))
   (segment (start 96.96 71.21) (end 97.64 71.21) (width 0.25) (layer "F.Cu") (net 6))
-  (segment (start 103.87 69.53) (end 104.79 69.53) (width 0.25) (layer "F.Cu") (net 6))
   (segment (start 104.75 70.28) (end 105.145 69.885) (width 0.25) (layer "F.Cu") (net 6))
   (segment (start 104.79 69.53) (end 105.145 69.885) (width 0.25) (layer "F.Cu") (net 6))
@@
   (via (at 94.91 75.28) (size 0.4) (drill 0.2) (layers "F.Cu" "B.Cu") (free) (net 6))
   (via (at 103.87 69.53) (size 0.4) (drill 0.2) (layers "F.Cu" "B.Cu") (free) (net 6))
-  (via (at 100.83 75.5) (size 0.4) (drill 0.2) (layers "F.Cu" "B.Cu") (free) (net 6))
+  (via (at 106.5 71.8) (size 0.4) (drill 0.2) (layers "F.Cu" "B.Cu") (free) (net 6))
+  (via (at 101 75.7) (size 0.4) (drill 0.2) (layers "F.Cu" "B.Cu") (free) (net 6))
+  (via (at 101.6 70.2) (size 0.4) (drill 0.2) (layers "F.Cu" "B.Cu") (free) (net 6))
+  (via (at 100.3 75.7) (size 0.4) (drill 0.2) (layers "F.Cu" "B.Cu") (free) (net 6))
+  (via (at 97.1 74.5) (size 0.4) (drill 0.2) (layers "F.Cu" "B.Cu") (free) (net 6))
+  (via (at 99 67.3) (size 0.4) (drill 0.2) (layers "F.Cu" "B.Cu") (free) (net 6))
   (via (at 108.64 71.79) (size 0.4) (drill 0.2) (layers "F.Cu" "B.Cu") (free) (net 6))
   (via (at 96.96 71.21) (size 0.4) (drill 0.2) (layers "F.Cu" "B.Cu") (free) (net 6))
   (via (at 108.37 67.67) (size 0.4) (drill 0.2) (layers "F.Cu" "B.Cu") (free) (net 6))
   (via (at 108.14 75.62) (size 0.4) (drill 0.2) (layers "F.Cu" "B.Cu") (free) (net 6))
+  (via (at 101 73.6) (size 0.4) (drill 0.2) (layers "F.Cu" "B.Cu") (free) (net 6))
   (via (at 103.23 68.02) (size 0.4) (drill 0.2) (layers "F.Cu" "B.Cu") (free) (net 6))
   (segment (start 102.9975 73.5) (end 102.445 74.0525) (width 0.25) (layer "F.Cu") (net 7))
@@
   (segment (start 99.61 72.26) (end 99.9 72.26) (width 0.25) (layer "F.Cu") (net 11))
   (zone (net 6) (net_name "GND2") (layer "F.Cu") (hatch edge 0.508)
-    (connect_pads (clearance 0.508))
+    (connect_pads thru_hole_only (clearance 0.508))
     (min_thickness 0.254) (filled_areas_thickness no)
     (fill yes (thermal_gap 0.508) (thermal_bridge_width 0.508))
@@
   )
   (zone (net 4) (net_name "GND1") (layer "F.Cu") (hatch edge 0.508)
-    (connect_pads (clearance 0.508))
+    (connect_pads thru_hole_only (clearance 0.508))
     (min_thickness 0.254) (filled_areas_thickness no)
     (fill yes (thermal_gap 0.508) (thermal_bridge_width 0.508))
