File: pcbs/logic_board_v1/timing_logic.kicad_sch (KiCad schematic)
At the start: 103 parts, among them J1 VCC, J2 VEE, J3 NIM_COINC, J4 NIM2, J5 NIM1, J6 Input1, J7 Input2, Q1 BFR92, Q2 BFR92, Q3 BFR92, Q4 BFR92, Q5 BFR92, Q6 BFR92, U1 8240026, U2 MAX9600EUP, U3 OPA177GP, U4 REF03GS, U5 MC100EP05DG

Commit message: Add files via upload
Parts:
- C1, C10, C11, C12, C13, C14, C15, C16, C17, C18, C19, C2, C20, C21, C3, C4, C5, C6, C7, C8, C9: footprint Capacitor_SMD:C_0201_0603Metric -> Capacitor_SMD:C_0603_1608Metric_Pad1.08x0.95mm_HandSolder
- R1, R10, R11, R12, R13, R14, R15, R16, R17, R18, R19, R2, R20, R21, R22, R23, R24, R25, R26, R27, R28, R29, R3, R30, R4, R5, R6, R7, R8, R9: footprint Resistor_SMD:R_0201_0603Metric -> Resistor_SMD:R_0603_1608Metric_Pad0.98x0.95mm_HandSolder
